Commit message: Updated F_soc, F_des by refering to global frame, modified F_soc with a better approach

File: install/differential_robot/share/differential_robot/urdf/diffbot_classic_gazebo.urdf (robot description, URDF)
Before this commit: robot diff_bot, 13 links, 12 joints
Joints:
- joint scan_joint: origin xyz=0.31 0 0.21 rpy=0 0 0 -> xyz=0.0 0 0.38 rpy=0 0 0
