Commit message: Added functions to calculate social forces from multiple human detections, created new human detections node, added social_force_calculator.py for testing social forces seperately...

File: src/differential_robot/urdf/diffbot_classic_gazebo.urdf (robot description, URDF)
Before this commit: robot diff_bot, 13 links, 12 joints
Joints:
- joint scan_joint: origin xyz=0.0 0 0.38 rpy=0 0 0 -> xyz=0.0 0 0.40 rpy=0 0 0
